Commit message: combine spot with gen3, also add some bounding boxes to let the operator know about other things on the spot

File: spot_description/urdf/spot_with_gen3.urdf.xacro (robot description, xacro)
@@ -355,5 +355,5 @@
     <!-- Front CB -->
     <link name="front_collision">
-    <!-- <visual>
+    <visual>
         <geometry>
         <box size="0.2 0.15 0.15" />
@@ -362,5 +362,5 @@
         <color rgba="1 0 0 1" />
         </material>
-    </visual> -->
+    </visual>
     <collision>
         <geometry>
@@ -376,5 +376,5 @@
     <!-- Back CB -->
     <link name="rear_collision">
-    <!-- <visual>
+    <visual>
         <geometry>
         <box size="0.4 0.15 0.15" />
@@ -383,5 +383,5 @@
         <color rgba="1 0 0 1" />
         </material>
-    </visual> -->
+    </visual>
     <collision>
         <geometry>

Commit message: Update spot_with_gen3.urdf.xacro
Updated bounding box for sensor board on arm

File: spot_description/urdf/spot_with_gen3.urdf.xacro (robot description, xacro)
@@ -395,4 +395,25 @@
         <origin xyz="-0.1 0 0.18" rpy="0 0 0" />
     </joint>
+    <!-- Arm sensor CB - height = 15 width = 10 lenght = 20 -->
+    <link name="readiness_sensor_collision">
+    <visual>
+        <geometry>
+        <box size="0.20 0.06 0.15" />
+        </geometry>
+        <material name="red">
+        <color rgba="0 0 1 1" />
+        </material>
+    </visual>
+    <collision>
+        <geometry>
+        <box size="0.20 0.06 0.15" />
+        </geometry>
+    </collision>
+    </link>
+    <joint name="readiness_sensor_collision_joint" type="fixed">
+        <child link="readiness_sensor_collision" />
+        <parent link="gen3_end_effector_link" />
+        <origin xyz="0.0 -0.07 0.0" rpy="0 0 0" />
+    </joint>
     <!-- Optional custom includes. -->
     <xacro:include filename="$(optenv SPOT_URDF_EXTRAS empty.urdf)" />

Commit message: sync with the nuc

File: spot_description/urdf/spot_with_gen3.urdf.xacro (robot description, xacro)
@@ -13,5 +13,5 @@
         </collision>
     </link>
-    <link name="base_link">
+    <!-- <link name="base_link">
         <inertial>
             <origin rpy="0.0 0.0 0.0" xyz="0.006394396536052227 -9.812158532440662e-05 0.0009113792330026627"/>
@@ -24,5 +24,5 @@
         <parent link="body" />
         <child link="base_link" />
-    </joint>
+    </joint> -->
     <link name="front_rail">
         <inertial>
@@ -343,14 +343,50 @@
     <xacro:arg name="dof" default="6" />
     <xacro:arg name="vision" default="true" />
+    <xacro:arg name="robot_ip" default="192.168.10.9" />
+    <xacro:arg name="username" default="admin" />
+    <xacro:arg name="password" default="admin" />
+    <xacro:arg name="port" default="10000" />
+    <xacro:arg name="port_realtime" default="10001" />
+    <xacro:arg name="session_inactivity_timeout_ms" default="60000" />
+    <xacro:arg name="connection_inactivity_timeout_ms" default="2000" />
     <xacro:arg name="gripper" default="robotiq_2f_140" />
-    <xacro:arg name="sim" default="false" />
-    <xacro:arg name="prefix" default="gen3_" />
-    <joint name="body_gen3" type="fixed">
-        <child link="$(arg prefix)base_link" />
-        <parent link="body" />
-        <origin xyz="0.1656 0 0.12" rpy="0 0 0" />
-    </joint>
+    <xacro:arg name="gripper_joint_name" default="finger_joint" />
+    <xacro:arg name="gripper_max_velocity" default="100.0" />
+    <xacro:arg name="gripper_max_force" default="100.0" />
+    <xacro:arg name="sim_gazebo" default="false" />
+    <xacro:arg name="sim_ignition" default="false" />
+    <xacro:arg name="sim_isaac" default="false" />
+    <xacro:arg name="prefix" default="" />
+    <xacro:arg name="use_fake_hardware" default="false" />
+    <xacro:arg name="fake_sensor_commands" default="false" />
+    <xacro:arg name="use_internal_bus_gripper_comm" default="true" />
+    <xacro:arg name="use_external_cable" default="false" />
     <xacro:include filename="$(find kortex_description)/robots/kortex_robot.xacro" />
-    <xacro:load_robot arm="$(arg arm)" gripper="$(arg gripper)" dof="$(arg dof)" vision="$(arg vision)" sim="$(arg sim)" prefix="$(arg prefix)"/>
+    <xacro:load_robot
+        parent="body"
+        arm="$(arg arm)"
+        gripper="$(arg gripper)"
+        gripper_joint_name="$(arg gripper_joint_name)"
+        gripper_max_velocity="$(arg gripper_max_velocity)"
+        gripper_max_force="$(arg gripper_max_force)"
+        dof="$(arg dof)"
+        vision="$(arg vision)"
+        robot_ip="$(arg robot_ip)"
+        username="$(arg username)"
+        password="$(arg password)"
+        port="$(arg port)"
+        port_realtime="$(arg port_realtime)"
+        session_inactivity_timeout_ms="$(arg session_inactivity_timeout_ms)"
+        connection_inactivity_timeout_ms="$(arg connection_inactivity_timeout_ms)"
+        use_internal_bus_gripper_comm="$(arg use_internal_bus_gripper_comm)"
+        prefix="$(arg prefix)"
+        use_fake_hardware="$(arg use_fake_hardware)"
+        fake_sensor_commands="$(arg fake_sensor_commands)"
+        sim_gazebo="$(arg sim_gazebo)"
+        sim_ignition="$(arg sim_ignition)"
+        sim_isaac="$(arg sim_isaac)"
+        use_external_cable="$(arg use_external_cable)" >
+        <origin xyz="0.1656 0 0.12" rpy="0 0 0" />  <!-- position robot in the world -->
+    </xacro:load_robot>
     <!-- Front CB -->
     <link name="front_collision">
@@ -395,6 +431,6 @@
         <origin xyz="-0.1 0 0.18" rpy="0 0 0" />
     </joint>
-    <!-- Arm sensor CB - height = 15 width = 10 lenght = 20 -->
-    <link name="readiness_sensor_collision">
+    <!-- Arm sensor CB - height = 15 width = 10 length = 20 -->
+    <!-- <link name="readiness_sensor_collision">
     <visual>
         <geometry>
@@ -415,5 +451,5 @@
         <parent link="gen3_end_effector_link" />
         <origin xyz="0.0 -0.07 0.0" rpy="0 0 0" />
-    </joint>
+    </joint> -->
     <!-- Optional custom includes. -->
     <xacro:include filename="$(optenv SPOT_URDF_EXTRAS empty.urdf)" />

Commit message: sync with the nuc

File: spot_description/urdf/spot_with_gen3.urdf.xacro (robot description, xacro)
@@ -408,5 +408,5 @@
         <child link="front_collision" />
         <parent link="body" />
-        <origin xyz="0.35 0 0.2" rpy="0 0 0" />
+        <origin xyz="0.35 0 0.15" rpy="0 0 0" />
     </joint>
     <!-- Back CB -->
@@ -414,5 +414,5 @@
     <visual>
         <geometry>
-        <box size="0.4 0.15 0.15" />
+        <box size="0.6 0.14 0.14" />
         </geometry>
         <material name="red">
@@ -422,5 +422,5 @@
     <collision>
         <geometry>
-        <box size="0.4 0.15 0.15" />
+        <box size="0.6 0.14 0.14" />
         </geometry>
     </collision>
@@ -429,5 +429,5 @@
         <child link="rear_collision" />
         <parent link="body" />
-        <origin xyz="-0.1 0 0.18" rpy="0 0 0" />
+        <origin xyz="-0.15 0 0.17" rpy="0 0 0" />
     </joint>
     <!-- Arm sensor CB - height = 15 width = 10 length = 20 -->
